Commit message: Add shoulder joints and arm_controller to nao_webots_driver

File: ros2_ws/src/nao_webots_driver/resource/nao_webots.urdf (robot description, URDF)
Before this commit: robot Nao Webots, 3 links, 2 joints
Links:
- added link l_shoulder_link
- added link l_upper_arm_link
- added link r_shoulder_link
- added link r_upper_arm_link
Joints:
- added joint LShoulderPitch: type revolute, parent base_link, child l_shoulder_link, origin xyz=0 0.1 0.1 rpy=0 0 0, axis 0 1 0, limit lower=-2.0857 upper=2.0857 effort=1.0 velocity=1.0
- added joint LShoulderRoll: type revolute, parent l_shoulder_link, child l_upper_arm_link, origin xyz=0 0 0 rpy=0 0 0, axis 1 0 0, limit lower=-0.3142 upper=1.3265 effort=1.0 velocity=1.0
- added joint RShoulderPitch: type revolute, parent base_link, child r_shoulder_link, origin xyz=0 -0.1 0.1 rpy=0 0 0, axis 0 1 0, limit lower=-2.0857 upper=2.0857 effort=1.0 velocity=1.0
- added joint RShoulderRoll: type revolute, parent r_shoulder_link, child r_upper_arm_link, origin xyz=0 0 0 rpy=0 0 0, axis 1 0 0, limit lower=-1.3265 upper=0.3142 effort=1.0 velocity=1.0

Commit message: Add elbow joints to nao_webots_drive

File: ros2_ws/src/nao_webots_driver/resource/nao_webots.urdf (robot description, URDF)
Before this commit: robot Nao Webots, 7 links, 6 joints
Links:
- added link l_elbow_link
- added link l_forearm_link
- added link r_elbow_link
- added link r_forearm_link
Joints:
- added joint LElbowRoll: type revolute, parent l_elbow_link, child l_forearm_link, origin xyz=0 0 0 rpy=0 0 0, axis 1 0 0, limit lower=-1.5446 upper=-0.0349 effort=1.0 velocity=1.0
- added joint LElbowYaw: type revolute, parent l_upper_arm_link, child l_elbow_link, origin xyz=0 0.1 0 rpy=0 0 0, axis 0 1 0, limit lower=-2.0857 upper=2.0857 effort=1.0 velocity=1.0
- added joint RElbowRoll: type revolute, parent r_elbow_link, child r_forearm_link, origin xyz=0 0 0 rpy=0 0 0, axis 1 0 0, limit lower=0.0349 upper=1.5446 effort=1.0 velocity=1.0
- added joint RElbowYaw: type revolute, parent r_upper_arm_link, child r_elbow_link, origin xyz=0 -0.1 0 rpy=0 0 0, axis 0 1 0, limit lower=-2.0857 upper=2.0857 effort=1.0 velocity=1.0
